Commit message: + urdf & meshes for rb

File: urdf/aubo_i5.urdf (robot description, URDF)
Before this commit: robot aubo_i5, 8 links, 7 joints
Links:
- removed link world
Joints:
- removed joint world_joint

File: urdf/aubo_i5.urdf.xacro (robot description, xacro)
@@ -5,7 +5,4 @@
 <!-- =================================================================================== -->
 <robot  name="aubo_i5" xmlns:xacro="http://www.ros.org/wiki/xacro">
-  <xacro:include filename="$(find aubo_description)/urdf/aubo.transmission.xacro" />
-  <xacro:include filename="$(find aubo_description)/urdf/aubo.gazebo.xacro" />
-  <xacro:include filename="$(find your_robot_description)/urdf/materials.xacro" />
   <link name="base_link">
     <inertial>
@@ -17,14 +14,14 @@
       <origin xyz="0 0 0" rpy="0 0 0" />
       <geometry>
-        <mesh filename="package://aubo_description/meshes/aubo_i5/visual/base_link.DAE" />
-      </geometry>
-      <material name="">
-        <color rgba="1 1 1 1" />
-      </material>
-    </visual>
-    <collision>
-      <origin xyz="0 0 0" rpy="0 0 0" />
-      <geometry>
-        <mesh filename="package://aubo_description/meshes/aubo_i5/collision/base_link.STL" />
+        <mesh filename="package://rb_description/meshes/aubo_i5/collision/base_link.STL" />
+      </geometry>
+      <material name="">
+        <color rgba="1 1 1 1" />
+      </material>
+    </visual>
+    <collision>
+      <origin xyz="0 0 0" rpy="0 0 0" />
+      <geometry>
+        <mesh filename="package://rb_description/meshes/aubo_i5/collision/base_link.STL" />
       </geometry>
     </collision>
@@ -39,14 +36,14 @@
       <origin xyz="0 0 0" rpy="0 0 0" />
       <geometry>
-        <mesh filename="package://aubo_description/meshes/aubo_i5/visual/shoulder_Link.DAE" />
-      </geometry>
-      <material name="">
-        <color rgba="1 1 1 1" />
-      </material>
-    </visual>
-    <collision>
-      <origin xyz="0 0 0" rpy="0 0 0" />
-      <geometry>
-        <mesh filename="package://aubo_description/meshes/aubo_i5/collision/shoulder_Link.STL" />
+        <mesh filename="package://rb_description/meshes/aubo_i5/collision/shoulder_Link.STL" />
+      </geometry>
+      <material name="">
+        <color rgba="1 1 1 1" />
+      </material>
+    </visual>
+    <collision>
+      <origin xyz="0 0 0" rpy="0 0 0" />
+      <geometry>
+        <mesh filename="package://rb_description/meshes/aubo_i5/collision/shoulder_Link.STL" />
       </geometry>
     </collision>
@@ -68,14 +65,14 @@
       <origin xyz="0 0 0" rpy="0 0 0" />
       <geometry>
-        <mesh filename="package://aubo_description/meshes/aubo_i5/visual/upperArm_Link.DAE" />
-      </geometry>
-      <material name="">
-        <color rgba="1 1 1 1" />
-      </material>
-    </visual>
-    <collision>
-      <origin xyz="0 0 0" rpy="0 0 0" />
-      <geometry>
-        <mesh filename="package://aubo_description/meshes/aubo_i5/collision/upperArm_Link.STL" />
+        <mesh filename="package://rb_description/meshes/aubo_i5/collision/upperArm_Link.STL" />
+      </geometry>
+      <material name="">
+        <color rgba="1 1 1 1" />
+      </material>
+    </visual>
+    <collision>
+      <origin xyz="0 0 0" rpy="0 0 0" />
+      <geometry>
+        <mesh filename="package://rb_description/meshes/aubo_i5/collision/upperArm_Link.STL" />
       </geometry>
     </collision>
@@ -97,14 +94,14 @@
       <origin xyz="0 0 0" rpy="0 0 0" />
       <geometry>
-        <mesh filename="package://aubo_description/meshes/aubo_i5/visual/foreArm_Link.DAE" />
-      </geometry>
-      <material name="">
-        <color rgba="1 1 1 1" />
-      </material>
-    </visual>
-    <collision>
-      <origin xyz="0 0 0" rpy="0 0 0" />
-      <geometry>
-        <mesh filename="package://aubo_description/meshes/aubo_i5/collision/foreArm_Link.STL" />
+        <mesh filename="package://rb_description/meshes/aubo_i5/collision/foreArm_Link.STL" />
+      </geometry>
+      <material name="">
+        <color rgba="1 1 1 1" />
+      </material>
+    </visual>
+    <collision>
+      <origin xyz="0 0 0" rpy="0 0 0" />
+      <geometry>
+        <mesh filename="package://rb_description/meshes/aubo_i5/collision/foreArm_Link.STL" />
       </geometry>
     </collision>
@@ -126,14 +123,14 @@
       <origin xyz="0 0 0" rpy="0 0 0" />
       <geometry>
-        <mesh filename="package://aubo_description/meshes/aubo_i5/visual/wrist1_Link.DAE" />
-      </geometry>
-      <material name="">
-        <color rgba="1 1 1 1" />
-      </material>
-    </visual>
-    <collision>
-      <origin xyz="0 0 0" rpy="0 0 0" />
-      <geometry>
-        <mesh filename="package://aubo_description/meshes/aubo_i5/collision/wrist1_Link.STL" />
+        <mesh filename="package://rb_description/meshes/aubo_i5/collision/wrist1_Link.STL" />
+      </geometry>
+      <material name="">
+        <color rgba="1 1 1 1" />
+      </material>
+    </visual>
+    <collision>
+      <origin xyz="0 0 0" rpy="0 0 0" />
+      <geometry>
+        <mesh filename="package://rb_description/meshes/aubo_i5/collision/wrist1_Link.STL" />
       </geometry>
     </collision>
@@ -155,14 +152,14 @@
       <origin xyz="0 0 0" rpy="0 0 0" />
       <geometry>
-        <mesh filename="package://aubo_description/meshes/aubo_i5/visual/wrist2_Link.DAE" />
-      </geometry>
-      <material name="">
-        <color rgba="1 1 1 1" />
-      </material>
-    </visual>
-    <collision>
-      <origin xyz="0 0 0" rpy="0 0 0" />
-      <geometry>
-        <mesh filename="package://aubo_description/meshes/aubo_i5/collision/wrist2_Link.STL" />
+        <mesh filename="package://rb_description/meshes/aubo_i5/collision/wrist2_Link.STL" />
+      </geometry>
+      <material name="">
+        <color rgba="1 1 1 1" />
+      </material>
+    </visual>
+    <collision>
+      <origin xyz="0 0 0" rpy="0 0 0" />
+      <geometry>
+        <mesh filename="package://rb_description/meshes/aubo_i5/collision/wrist2_Link.STL" />
       </geometry>
     </collision>
@@ -184,14 +181,14 @@
       <origin xyz="0 0 0" rpy="0 0 0" />
       <geometry>
-        <mesh filename="package://aubo_description/meshes/aubo_i5/visual/wrist3_Link.DAE" />
-      </geometry>
-      <material name="">
-        <color rgba="1 1 1 1" />
-      </material>
-    </visual>
-    <collision>
-      <origin xyz="0 0 0" rpy="0 0 0" />
-      <geometry>
-        <mesh filename="package://aubo_description/meshes/aubo_i5/collision/wrist3_Link.STL" />
+        <mesh filename="package://rb_description/meshes/aubo_i5/collision/wrist3_Link.STL" />
+      </geometry>
+      <material name="">
+        <color rgba="1 1 1 1" />
+      </material>
+    </visual>
+    <collision>
+      <origin xyz="0 0 0" rpy="0 0 0" />
+      <geometry>
+        <mesh filename="package://rb_description/meshes/aubo_i5/collision/wrist3_Link.STL" />
       </geometry>
     </collision>
@@ -204,9 +201,3 @@
     <limit lower="-3.05" upper="3.05" effort="0" velocity="0" />
   </joint>
-  <link name="world" />
-  <joint name="world_joint" type="fixed">
-    <parent link="world" />
-    <child link = "base_link" />
-    <origin xyz="0.0 0.0 0.0" rpy="0.0 0.0 0.0" />
-  </joint>
 </robot>

File: urdf/aubo_i5_robot.urdf.xacro (robot description, xacro)
@@ -4,11 +4,10 @@
   <!-- Aubo -->
   <xacro:include filename="$(find rb_description)/urdf/aubo_i5.urdf.xacro" />
-  <xacro:xarm7_urdf prefix="" />
   <!-- Moving platform -->
   <xacro:include filename="$(find rb_description)/urdf/platform.urdf.xacro"/>
   <joint name="manipulator_joint" type="fixed">
-    <parent link="base_platform_base_link"/>
+    <parent link="robot_barmen_base_link"/>
     <child link="base_link"/>
-    <origin xyz="0.25 0.00 0.458" rpy="0 0 0"/>
+    <origin xyz="0.0 0.25 0.458" rpy="0 0 0"/>
   </joint>
 </robot>

File: urdf/platform.urdf.xacro (robot description, xacro)
@@ -1,7 +1,5 @@
 <?xml version="1.0"?>
 <robot name="base_platform" xmlns:xacro="http://ros.org/wiki/xacro">
-    <xacro:property name="prefix" value="base_platform_"/>
-    <xacro:include filename="$(find rb_description)/urdf/macros.xacro"/>
-    <link name="${prefix}base_link">
+    <link name="robot_barmen_base_link">
         <visual>
             <geometry>
