Commit message: + rb description

File: urdf/aubo_i5_robot.urdf.xacro (robot description, xacro)
@@ -1,16 +1,14 @@
 <?xml version="1.0"?>
-<robot xmlns:xacro="http://ros.org/wiki/xacro"
-       name="aubo_i5" >
-  <!-- common stuff -->
-  <xacro:include filename="$(find aubo_description)/urdf/common.gazebo.xacro" />
-  <!-- ur5 -->
-  <xacro:include filename="$(find aubo_description)/urdf/aubo_i5.urdf.xacro" />
-  <!-- arm -->
-  <xacro:aubo_i5L_robot prefix="" joint_limited="false"/>
-  <link name="world" />
-  <joint name="world_joint" type="fixed">
-    <parent link="world" />
-    <child link = "base_link" />
-    <origin xyz="0.0 0.0 0.0" rpy="0.0 0.0 0.0" />
+<robot xmlns:xacro="http://ros.org/wiki/xacro" name="robot_cleaner">
+  <xacro:arg name="fixed_base" default="false"/>
+  <!-- Aubo -->
+  <xacro:include filename="$(find rb_description)/urdf/aubo_i5.urdf.xacro" />
+  <xacro:xarm7_urdf prefix="" />
+  <!-- Moving platform -->
+  <xacro:include filename="$(find rb_description)/urdf/platform.urdf.xacro"/>
+  <joint name="manipulator_joint" type="fixed">
+    <parent link="base_platform_base_link"/>
+    <child link="base_link"/>
+    <origin xyz="0.25 0.00 0.458" rpy="0 0 0"/>
   </joint>
 </robot>

Commit message: + rb model fixing

File: urdf/aubo_i5_robot.urdf.xacro (robot description, xacro)
@@ -9,5 +9,5 @@
     <parent link="robot_barmen_base_link"/>
     <child link="base_link"/>
-    <origin xyz="0.0 0.25 0.458" rpy="0 0 0"/>
+    <origin xyz="0.25 0.0 0.458" rpy="0 0 0"/>
   </joint>
 </robot>

Commit message: + gripper done

File: urdf/aubo_i5_robot.urdf.xacro (robot description, xacro)
@@ -6,8 +6,16 @@
   <!-- Moving platform -->
   <xacro:include filename="$(find rb_description)/urdf/platform.urdf.xacro"/>
-  <joint name="manipulator_joint" type="fixed">
+  <joint name="robot_base_joint" type="fixed">
     <parent link="robot_barmen_base_link"/>
     <child link="base_link"/>
     <origin xyz="0.25 0.0 0.458" rpy="0 0 0"/>
   </joint>
+  <!-- Gripper -->
+  <xacro:include filename="$(find rb_description)/urdf/gripper.urdf.xacro"/>
+  <joint name="manipulator_joint" type="fixed">
+    <parent link="wrist3_Link"/>
+    <child link="robot_barmen_gripper_link"/>
+    <origin xyz="0 0 0" rpy="0 0 0"/>
+    <axis xyz="0 0 1"/>
+  </joint>
 </robot>
