Commit message: + gripper new offset

File: urdf/gripper.urdf.xacro (robot description, xacro)
@@ -6,5 +6,5 @@
                 <mesh filename="package://rb_description/meshes/gripper.stl"/>
             </geometry>
-            <origin xyz="-0.0025 0.0 0.16" rpy="0 0 0"/>
+            <origin xyz="-0.0025 0.0 0.214" rpy="0 0 0"/>
             <material name="blue"/>
         </visual>
